File: simpleCh552/simpleCh552.kicad_pcb (KiCad board)
At the start: 2 copper layers, 109.3 x 40 mm, 15 parts, among them J1 Conn_01x04, J5 Conn_01x06, J6 Conn_01x06, SW1 SW_SPST, U1 CH552G

Commit message: update
Parts:
- moved RV1 110.0 mm to (190.9, 97.6), turned to 45 degrees
- moved J5 97.2 mm to (184.8, 97.0), turned to 180 degrees
- moved RV2 94.5 mm to (183.8, 119.3), turned to -45 degrees
- moved RV3 86.9 mm to (161.7, 112.5)
- moved RV4 62.0 mm to (168.9, 90.0), turned to 135 degrees
Routing:
- net Net-(J5-Pin_2): track 16.0 -> 7.38 mm
- net Net-(J5-Pin_5): track 11.2 -> 6.52 mm
- net VSS: track 104.9 -> 109.5 mm
- net Net-(J5-Pin_3): track 19.4 -> 22.8 mm
- net Net-(J5-Pin_4): track 19.6 -> 22.7 mm
Other:
- board size 109.3 x 40 mm -> 40 x 76.9 mm
